Commit message: TRAVERSER: Enabling Gazebo simulation with the traverser

File: robots/traverser/description/urdf/actuators/wheel.urdf.xacro (robot description, xacro)
@@ -3,7 +3,8 @@
 <robot xmlns:xacro="http://www.ros.org/wiki/xacro">
     <xacro:macro name="wheel" params="name parent *origin
+                                      length:=0.05
+                                      radius:=0.05
                                       material_name:=black
-                                      length:=0.05
-                                      radius:=0.05">
+                                      gazebo_material_name:=Gazebo/Black">
         <joint name="${parent}_to_${name}_wheel_joint" type="continuous">
             <axis xyz="0 0 1"/>
@@ -25,4 +26,7 @@
             </collision>
         </link>
+        <gazebo reference="${name}_wheel_link">
+            <material>${gazebo_material_name}</material>
+        </gazebo>
     </xacro:macro>
 </robot>

File: robots/traverser/description/urdf/traverser.urdf.xacro (robot description, xacro)
@@ -8,5 +8,7 @@
                                           wheel_thickness:=0.05
                                           wheel_radius:=0.05
-                                          wheel_height:=0.025">
+                                          wheel_height:=0.025
+                                          gazebo_platform_material:=Gazebo/Blue
+                                          gazebo_wheel_material:=Gazebo/Black">
         <!-- Include xacro files-->
         <xacro:include filename="$(find robot_common)/urdf/common.urdf.xacro" />
@@ -39,8 +41,12 @@
                                   height="${platform_height}" />
         </link>
+        <gazebo reference="${name}_link">
+            <material>${gazebo_platform_material}</material>
+        </gazebo>
         <!-- Wheels -->
         <xacro:wheel name="right_front" parent="${name}_link"
                      length="${wheel_thickness}" radius="${wheel_radius}"
-                     material_name="black">
+                     material_name="black"
+                     gazebo_material_name="${gazebo_wheel_material}">
             <origin xyz="${(platform_length/2)-wheel_radius}
                          ${-1*((platform_width/2)+(wheel_thickness/2))}
@@ -50,5 +56,6 @@
         <xacro:wheel name="left_front" parent="${name}_link"
                      length="${wheel_thickness}" radius="${wheel_radius}"
-                     material_name="black">
+                     material_name="black"
+                     gazebo_material_name="${gazebo_wheel_material}">
             <origin xyz="${(platform_length/2)-wheel_radius}
                          ${1*((platform_width/2)+(wheel_thickness/2))}
@@ -58,5 +65,6 @@
         <xacro:wheel name="right_back" parent="${name}_link"
                      length="${wheel_thickness}" radius="${wheel_radius}"
-                     material_name="black">
+                     material_name="black"
+                     gazebo_material_name="${gazebo_wheel_material}">
             <origin xyz="${-1*((platform_length/2)-wheel_radius)}
                          ${-1*((platform_width/2)+(wheel_thickness/2))}
@@ -66,5 +74,6 @@
         <xacro:wheel name="left_back" parent="${name}_link"
                      length="${wheel_thickness}" radius="${wheel_radius}"
-                     material_name="black">
+                     material_name="black"
+                     gazebo_material_name="${gazebo_wheel_material}">
             <origin xyz="${-1*((platform_length/2)-wheel_radius)}
                          ${1*((platform_width/2)+(wheel_thickness/2))}

File: robots/traverser/description/variants/traverser.urdf.xacro (robot description, xacro)
@@ -10,6 +10,6 @@
                      wheel_radius="${traverser_wheel_radius}">
         <!--This defines the co-ordinate transform from base_body to base_link -->
-        <!-- base link is on ground z = 0 and base_body_link is offset to z = `traverser_wheel_radius`.
-             ROS Nav needs a frame at axis of rotation on ground, which in our case is base_link -->
+        <!--base link is on ground z = 0 and base_body_link is offset to z = `traverser_wheel_radius`.
+            ROS Nav needs a frame at axis of rotation on ground, which in our case is base_link -->
         <origin xyz="0 0 ${traverser_wheel_radius}" rpy="0 0 0" />
     </xacro:traverser>

Commit message: TRAVERSER: Fix to spawn complete robot (with wheels) in Gazebo.

File: robots/traverser/description/urdf/actuators/wheel.urdf.xacro (robot description, xacro)
@@ -25,8 +25,19 @@
                 </geometry>
             </collision>
+            <xacro:cylinder_inertia mass="12" radius="${radius}"
+                                    length="${length}" />
         </link>
         <gazebo reference="${name}_wheel_link">
             <material>${gazebo_material_name}</material>
         </gazebo>
+        <!-- <transmission name="${name}_wheel_link">
+            <type>transmission_interface/SimpleTransmission</type>
+            <joint name="${parent}_to_${name}_wheel_joint">
+                <hardwareInterface>hardware_interface/VelocityJointInterface</hardwareInterface>
+            </joint>
+            <actuator name="${name}_wheel_motor">
+                <mechanicalReduction>1</mechanicalReduction>
+            </actuator>
+        </transmission> -->
     </xacro:macro>
 </robot>

File: robots/traverser/description/variants/traverser.urdf.xacro (robot description, xacro)
@@ -4,4 +4,5 @@
     <!-- Include xacro files-->
     <xacro:include filename="$(find robot_common)/urdf/materials.urdf.xacro" />
+    <xacro:include filename="$(find robot_common)/urdf/gazebo_ros_control.urdf.xacro" />
     <xacro:include filename="$(find traverser)/description/urdf/traverser.urdf.xacro" />
     <link name="base_link" />

Commit message: TRAVERSER: Added dynamic mass calculation and friction params

File: robots/traverser/description/urdf/actuators/wheel.urdf.xacro (robot description, xacro)
@@ -7,4 +7,7 @@
                                       material_name:=black
                                       gazebo_material_name:=Gazebo/Black">
+        <xacro:property name="wheel_density" value="1522.0"/> <!-- rubber -->
+        <xacro:property name="wheel_mass"
+                        value="${wheel_density * pi * radius * radius * length}"/>
         <joint name="${parent}_to_${name}_wheel_joint" type="continuous">
             <axis xyz="0 0 1"/>
@@ -25,9 +28,15 @@
                 </geometry>
             </collision>
-            <xacro:cylinder_inertia mass="12" radius="${radius}"
+            <xacro:cylinder_inertia mass="${wheel_mass}" radius="${radius}"
                                     length="${length}" />
         </link>
         <gazebo reference="${name}_wheel_link">
             <material>${gazebo_material_name}</material>
+            <mu1>1.0</mu1>
+            <mu2>1.0</mu2>
+            <kp>1000000.0</kp> <!-- kp and kd for rubber -->
+            <kd>100.0</kd>
+            <maxVel>1.0</maxVel>
+            <minDepth>0.00</minDepth>
         </gazebo>
         <!-- <transmission name="${name}_wheel_link">

File: robots/traverser/description/urdf/traverser.urdf.xacro (robot description, xacro)
@@ -14,4 +14,7 @@
         <xacro:include filename="$(find robot_common)/urdf/common.urdf.xacro" />
         <xacro:include filename="$(find traverser)/description/urdf/actuators/wheel.urdf.xacro" />
+        <xacro:property name="platform_density" value="7850.0"/> <!-- steel -->
+        <xacro:property name="platform_mass"
+                        value="${platform_density * platform_length * platform_width * platform_height}"/>
         <gazebo>
             <plugin name="skid_steer_drive_controller" filename="libgazebo_ros_skid_steer_drive.so">
@@ -27,7 +30,7 @@
                 <torque>20</torque>
                 <broadcastTF>true</broadcastTF>
-                <commandTopic>/cmd_vel</commandTopic>
-                <odometryTopic>/odom</odometryTopic>
-                <odometryFrame>/odom</odometryFrame>
+                <commandTopic>cmd_vel</commandTopic>
+                <odometryTopic>odom</odometryTopic>
+                <odometryFrame>odom</odometryFrame>
                 <covariance_x>0.0001</covariance_x>
                 <covariance_y>0.0001</covariance_y>
@@ -58,5 +61,5 @@
                 <origin rpy="0 0 0" xyz="0 0 ${(platform_height/2)-wheel_height}"/>
             </collision>
-            <xacro:cuboid_inertia mass="12" length="${platform_length}"
+            <xacro:cuboid_inertia mass="${platform_mass}" length="${platform_length}"
                                   breadth="${platform_width}"
                                   height="${platform_height}" />

Commit message: TRAVERSER: Added gazebo plugin and using it in traverser instead of skid steer

File: robots/traverser/description/urdf/actuators/wheel.urdf.xacro (robot description, xacro)
@@ -33,20 +33,7 @@
         <gazebo reference="${name}_wheel_link">
             <material>${gazebo_material_name}</material>
-            <mu1>1.0</mu1>
-            <mu2>1.0</mu2>
-            <kp>1000000.0</kp> <!-- kp and kd for rubber -->
-            <kd>100.0</kd>
-            <maxVel>1.0</maxVel>
-            <minDepth>0.00</minDepth>
+            <mu1>0.0</mu1>
+            <mu2>0.0</mu2>
         </gazebo>
-        <!-- <transmission name="${name}_wheel_link">
-            <type>transmission_interface/SimpleTransmission</type>
-            <joint name="${parent}_to_${name}_wheel_joint">
-                <hardwareInterface>hardware_interface/VelocityJointInterface</hardwareInterface>
-            </joint>
-            <actuator name="${name}_wheel_motor">
-                <mechanicalReduction>1</mechanicalReduction>
-            </actuator>
-        </transmission> -->
     </xacro:macro>
 </robot>

File: robots/traverser/description/urdf/traverser.urdf.xacro (robot description, xacro)
@@ -18,22 +18,10 @@
                         value="${platform_density * platform_length * platform_width * platform_height}"/>
         <gazebo>
-            <plugin name="skid_steer_drive_controller" filename="libgazebo_ros_skid_steer_drive.so">
-                <updateRate>50.0</updateRate>
-                <robotNamespace>/</robotNamespace>
-                <leftFrontJoint>base_body_link_to_left_front_wheel_joint</leftFrontJoint>
-                <rightFrontJoint>base_body_link_to_right_front_wheel_joint</rightFrontJoint>
-                <leftRearJoint>base_body_link_to_left_back_wheel_joint</leftRearJoint>
-                <rightRearJoint>base_body_link_to_right_back_wheel_joint</rightRearJoint>
-                <wheelSeparation>${platform_width + wheel_thickness}</wheelSeparation>
-                <wheelDiameter>${2*wheel_radius}</wheelDiameter>
-                <robotBaseFrame>${parent}</robotBaseFrame>
-                <torque>20</torque>
-                <broadcastTF>true</broadcastTF>
-                <commandTopic>cmd_vel</commandTopic>
-                <odometryTopic>odom</odometryTopic>
-                <odometryFrame>odom</odometryFrame>
-                <covariance_x>0.0001</covariance_x>
-                <covariance_y>0.0001</covariance_y>
-                <covariance_yaw>0.01</covariance_yaw>
+            <plugin name="traverser_controller" filename="libtraverser_controller_plugin.so">
+                <commandTopic>/cmd_vel</commandTopic>
+                <odometryTopic>/odom</odometryTopic>
+                <odometryFrame>/odom</odometryFrame>
+                <odometryRate>20.0</odometryRate>
+                <robotBaseFrame>/base_link</robotBaseFrame>
             </plugin>
         </gazebo>
